Commit message: Gazebo simulation of a simple robot

File: src/mybot_description/urdf/mybot.xacro (robot description, xacro)
@@ -52,5 +52,4 @@
   </link>
   <link name="left_wheel">
-    <!--origin xyz="0.1 0.13 0.1" rpy="0 1.5707 1.5707"/-->
     <collision name="collision">
       <origin xyz="0 0 0" rpy="0 1.5707 1.5707"/>
@@ -76,5 +75,4 @@
   </link>
   <link name="right_wheel">
-    <!--origin xyz="0.1 -0.13 0.1" rpy="0 1.5707 1.5707"/-->
     <collision name="collision">
       <origin xyz="0 0 0" rpy="0 1.5707 1.5707"/>
@@ -101,5 +99,4 @@
   <joint type="continuous" name="left_wheel_hinge">
     <origin xyz="0.1 0.15 0" rpy="0 0 0"/>
-    <!--origin xyz="0.1 0.13 0" rpy="0 1.5707 1.5707"/-->
     <child link="left_wheel"/>
     <parent link="chassis"/>
@@ -117,5 +114,5 @@
     <joint_properties damping="0.0" friction="0.0"/>
   </joint>
-  <link name="camera">
+  <link name="tof">
     <collision>
       <origin xyz="0 0 0" rpy="0 0 0"/>
@@ -142,31 +139,5 @@
     <origin xyz=".2 0 0" rpy="0 0 0"/>
     <parent link="chassis"/>
-    <child link="camera"/>
+    <child link="tof"/>
   </joint>
-  <joint name="hokuyo_joint" type="fixed">
-    <axis xyz="0 1 0" />
-    <origin xyz=".15 0 .1" rpy="0 0 0"/>
-    <parent link="chassis"/>
-    <child link="hokuyo"/>
-  </joint>
-  <!-- Hokuyo Laser -->
-  <link name="hokuyo">
-    <collision>
-      <origin xyz="0 0 0" rpy="0 0 0"/>
-      <geometry>
-    <box size="0.1 0.1 0.1"/>
-      </geometry>
-    </collision>
-    <visual>
-      <origin xyz="0 0 0" rpy="0 0 0"/>
-      <geometry>
-        <mesh filename="package://mybot_description/meshes/hokuyo.dae"/>
-      </geometry>
-    </visual>
-    <inertial>
-      <mass value="1e-5" />
-      <origin xyz="0 0 0" rpy="0 0 0"/>
-      <inertia ixx="1e-6" ixy="0" ixz="0" iyy="1e-6" iyz="0" izz="1e-6" />
-    </inertial>
-  </link>
 </robot>

Commit message: Some minor changes on robot

File: src/mybot_description/urdf/mybot.xacro (robot description, xacro)
@@ -7,8 +7,7 @@
   <xacro:include filename="$(find mybot_description)/urdf/macros.xacro" />
   <link name='chassis'>
-    <pose>0 0 0.1 0 0 0</pose>
     <inertial>
       <mass value="10.0"/>
-      <origin xyz="0.0 0 0.1" rpy=" 0 0 0"/>
+      <origin xyz="0.0 0 0.2" rpy=" 0 0 0"/>
       <inertia
           ixx="0.5" ixy="0" ixz="0"
@@ -19,5 +18,5 @@
     <collision name='collision'>
       <geometry>
-        <box size=".4 .2 .1"/>
+        <box size=".4 .2 .2"/>
       </geometry>
     </collision>
@@ -25,9 +24,9 @@
       <origin xyz="0 0 0" rpy=" 0 0 0"/>
       <geometry>
-        <box size=".4 .2 .1"/>
+        <box size=".4 .2 .2"/>
       </geometry>
     </visual>
     <collision name='caster_collision'>
-      <origin xyz="-0.15 0 -0.05" rpy=" 0 0 0"/>
+      <origin xyz="-0.15 0 -0.10" rpy=" 0 0 0"/>
       <geometry>
         <sphere radius="0.05"/>
@@ -45,5 +44,5 @@
     </collision>
     <visual name='caster_visual'>
-      <origin xyz="-0.15 0 -0.05" rpy=" 0 0 0"/>
+      <origin xyz="-0.15 0 -0.10" rpy=" 0 0 0"/>
       <geometry>
         <sphere radius="0.05"/>
@@ -98,5 +97,5 @@
   </link>
   <joint type="continuous" name="left_wheel_hinge">
-    <origin xyz="0.1 0.15 0" rpy="0 0 0"/>
+    <origin xyz="0.1 0.15 -0.05" rpy="0 0 0"/>
     <child link="left_wheel"/>
     <parent link="chassis"/>
@@ -106,5 +105,5 @@
   </joint>
   <joint type="continuous" name="right_wheel_hinge">
-    <origin xyz="0.1 -0.15 0" rpy="0 0 0"/>
+    <origin xyz="0.1 -0.15 -0.05" rpy="0 0 0"/>
     <!--origin xyz="0.1 -0.13 0" rpy="0 1.5707 1.5707"/-->
     <child link="right_wheel"/>
@@ -137,5 +136,5 @@
   <joint name="camera_joint" type="fixed">
     <axis xyz="0 1 0" />
-    <origin xyz=".2 0 0" rpy="0 0 0"/>
+    <origin xyz=".2 0 .12" rpy="0 0 0"/>
     <parent link="chassis"/>
     <child link="tof"/>
